Commit message: payload distributor

File: rotors_description/urdf/collaborative/four_hummingbirds_payload.xacro (robot description, xacro)
@@ -29,5 +29,5 @@
 	  <xacro:property name="payload_width" value="2.0" />
 	  <xacro:property name="payload_height" value="0.1" />
-	  <xacro:property name="payload_mass" value="0.01" />
+	  <xacro:property name="payload_mass" value="1.0" />
 	  <xacro:property name="payload_name" value="payload" />
 	  <xacro:property name="holder_width" value ="0.1" />

Commit message: modifications

File: rotors_description/urdf/collaborative/four_hummingbirds_payload.xacro (robot description, xacro)
@@ -33,5 +33,5 @@
 	  <xacro:property name="holder_width" value ="0.1" />
 	  <xacro:property name="holder_height" value="0.2" />
-	  <xacro:property name="mass_holder" value="0.1" />
+	  <xacro:property name="mass_holder" value="1.0" />
 	<xacro:include filename="$(find rotors_description)/urdf/collaborative/component_snippets.xacro" />
 	<xacro:include filename="$(find rotors_description)/urdf/collaborative/hummingbird_payload_offset.xacro"/>
